File: BOOSTV2.kicad_pcb (KiCad board)
At the start: 2 copper layers, 100 x 100 mm, 195 parts, among them IC1 ESDALC6V1W5, J1 PHNX_CONN_1017521, J2 PHNX_CONN_1017521, J3 USB_C_Receptacle_USB2.0_14P, J4 STM32-Prog-Header, J5 OLED, Q1 SI2302A-TPMSCT-ND, Q2 SI2302A-TPMSCT-ND, Q3 SI2302A-TPMSCT-ND, Q4 SI2302A-TPMSCT-ND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

Commit message: made repo
Parts:
- removed kibuzzard-67B59132: G***, kibuzzard-67B59132
- added kibuzzard-69165839: G***, kibuzzard-69165839, F.Cu at (160.4, 123.4)
