File: DC-Boost Hardware/BOOSTV2/EnablePin.kicad_sch (KiCad schematic)
At the start: 2 parts

Commit message: update
Other:
- company: (none) -> EcoCar
Changed lines of the file:
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@@
 (kicad_sch
-	(version 20231120)
+	(version 20250114)
 	(generator "eeschema")
-	(generator_version "8.0")
+	(generator_version "9.0")
 	(paper "A4")
 	(title_block
-		(comment 1 "Designed by: Nicholas semmens, Zeeshan Haque")
+		(rev "V2")
+		(company "EcoCar")
+		(comment 1 "Designed by:  Zeeshan Haque")
 	)
 	(junction
@@
 		(shape output)
 		(at 173.99 82.55 0)
-		(fields_autoplaced yes)
 		(effects
 			(font
@@
 		(shape input)
 		(at 109.855 82.55 180)
-		(fields_autoplaced yes)
 		(effects
 			(font
