File: DC-Boost Hardware/BOOSTV2/BOOSTV2.kicad_pcb (KiCad board)
At the start: 2 copper layers, 100 x 100 mm, 195 parts, among them IC1 ESDALC6V1W5, J1 PHNX_CONN_1017521, J2 PHNX_CONN_1017521, J3 USB_C_Receptacle_USB2.0_14P, J4 STM32-Prog-Header, J5 OLED, Q1 SI2302A-TPMSCT-ND, Q2 SI2302A-TPMSCT-ND, Q3 SI2302A-TPMSCT-ND, Q4 SI2302A-TPMSCT-ND, SW1 SW_SPDT, SW2 SW_SPDT, SW3 RESET, SW4 O/P Voltage Adjust, U1 ACS713xLCTR-30A, U10 NTMFS4D0N08XT1G, U11 NTMFS4D0N08XT1G, U12 ACS713xLCTR-30A, U13 MCP2542FD, U14 STM32G491KEUx, U15 AZ1117IH-5.0, U16 AZ1117IH-3.3, U17 TPS259631, U18 TPS259631, U2 MCP6007, U20 MCP6007, U3 LM51231QRGRRQ1, U4 NTMFS4D0N08XT1G, U5 NTMFS4D0N08XT1G, U6 NTMFS4D0N08XT1G, U7 NTMFS4D0N08XT1G, U8 NTMFS4D0N08XT1G, U9 NTMFS4D0N08XT1G, X1 OXETDLJANF-8MHZ

Commit message: update
Parts:
- removed kibuzzard-67B59132: G***, kibuzzard-67B59132
- added kibuzzard-694391D4: G***, kibuzzard-694391D4, F.Cu at (160.5, 123.2)

Commit message: update
Parts:
- removed kibuzzard-694391D4: G***, kibuzzard-694391D4
- added kibuzzard-694398FD: G***, kibuzzard-694398FD, F.Cu at (160.5, 123.2)
