File: DC-Boost Hardware/BOOSTV3/BOOSTV3.kicad_sch (KiCad schematic)
At the start: 6 parts

Commit message: update
Parts:
- added FID1, FID2, FID3, FID4, FID5, FID6: Fiducial, Fiducial:Fiducial_1mm_Mask2mm, symbol Mechanical:Fiducial
