File: DC-Boost Hardware/BOOSTV3/boost_circuit.kicad_sch (KiCad schematic)
At the start: 65 parts, among them J1 PHNX_CONN_1017521, J2 PHNX_CONN_1017521, SW1 SW_SPDT, SW2 SW_SPDT, U1 ACS713xLCTR-30A, U10 NTMFS4D0N08XT1G, U11 NTMFS4D0N08XT1G, U12 ACS713xLCTR-30A, U2 MCP6007, U3 LM51231QRGRRQ1, U4 NTMFS4D0N08XT1G, U5 NTMFS4D0N08XT1G, U6 NTMFS4D0N08XT1G, U7 NTMFS4D0N08XT1G, U8 NTMFS4D0N08XT1G, U9 NTMFS4D0N08XT1G

Commit message: update
Parts:
- removed J1, J2: PHNX_CONN_1017521, ecocad_lib_footprints:PHOENIX_1017521, symbol ecocad_lib_symbols:PHNX_CONN_1017521
- removed JP2: SolderJumper_2_Open, Jumper:SolderJumper-2_P1.3mm_Open_RoundedPad1.0x1.5mm, symbol Jumper:SolderJumper_2_Open
- added U21, U22: ~, ecocad_lib_footprints:PowerPole15-45BoardEdge2x1, symbol ecocad_lib_symbols:PowerPole2x1
- C11: value 47u -> 330n
- C12: value 220p -> 100p
- C14: value 12n -> 15n
- L1: value 2.2u -> 1.461u; footprint ecocad_lib_footprints:L_Kemet_3u3 -> ecocad_lib_footprints:3u3_induc
- R11: value 0.750u -> 722u; footprint ecocad_lib_footprints:CSS2H3920RL700F -> ecocad_lib_footprints:1u5_res_; DK Part # CSSH0805FT1L50 -> Y14840R00150F9R
- R4: value 15.4k -> 13k
Connections:
- net GNDREF is gone; now on net GND: C1.2, C10.2, C13.1, C19.2, C2.2, C20.2, C21.2, C22.2, C23.2, C24.2, C25.2, C26.2, C27.2, C28.2, C29.2, C3.2, C30.2, C31.2, C32.1, C4.2, C5.2, C6.2, C7.2, C8.2, C9.2, NT1.1, U1.5 (GND), U10.1 (S), U10.2 (S), U10.3 (S), U12.5 (GND), U3.10 (PGND), U3.19 (AGND), U3.21 (EP), U4.1 (S), U4.2 (S), U4.3 (S), U6.1 (S), U6.2 (S), U6.3 (S), U8.1 (S), U8.2 (S), U8.3 (S)
- net CSN: now also L1.2; no longer L1.1
- net GND: now also U21.1, U22.2
- net Low_Fets: now also L1.1; no longer L1.2
- net VOLT_IN_1: now also U21.2
- net VOLT_IN_2: now also U22.1
Other:
- note removed: "Equivalent to 198 uF"
- moved on the sheet: C1, C10, C11, C12, C13, C14, C15, C17, C18, C19, C2, C20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
