File: DC-Boost Hardware/BOOSTV3/mcu.kicad_sch (KiCad schematic)
At the start: 87 parts, among them IC1 ESDALC6V1W5, J3 USB_C_Receptacle_USB2.0_14P, J4 STM32-Prog-Header, J5 OLED, Q1 SI2302A-TPMSCT-ND, Q2 SI2302A-TPMSCT-ND, Q3 SI2302A-TPMSCT-ND, Q4 SI2302A-TPMSCT-ND, SW3 RESET, SW4 O/P Voltage Adjust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

Commit message: update
Other:
- note removed: "ESD Protected CAN Tranciever"
Changed lines of the file:
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@@
 	(title_block
 		(title "Microcontroller")
-		(rev "V2")
+		(rev "V3")
 		(company "EcoCar")
 		(comment 1 "Designed by:  Zeeshan Haque")
@@
 	(text "        V_{UVLO(F)} = (R2 + R3)/(R1 + R2 + R3) * V_{IN(UV)}\nV_{OVLO(F)} = R3/(R1 + R2 + R3) * V_{IN(OV)}\n\nV_{UVLO,F} from datasheet\n\n"
 		(exclude_from_sim no)
-		(at 175.26 275.59 0)
+		(at 175.895 275.59 0)
 		(effects
 			(font
@@
 	(text "LDO requires voltage drop of at least 1.3V\nMake undervoltage condition ~5V to ensure 3.3V V_{out} "
 		(exclude_from_sim no)
-		(at 234.315 274.955 0)
+		(at 236.22 276.225 0)
 		(effects
 			(font
@@
 		)
 	)
-	(text "ESD Protected CAN Tranciever\n"
-		(exclude_from_sim no)
-		(at 113.919 199.009 0)
-		(effects
-			(font
-				(size 1.27 1.27)
-			)
-			(justify right bottom)
-		)
-	)
 	(text "This IC features reverse polarity protection, current\nlimiting, UVLO and OVLO as well as a ~{FAULT} to detect\nfault conditions via an LED in our purpose."
 		(exclude_from_sim no)
@@
 	(text "eFuses FLT Circuitry\n"
 		(exclude_from_sim no)
-		(at 287.655 150.495 0)
-		(effects
-			(font
+		(at 290.83 146.05 0)
+		(effects
+			(font
